Commit message: Add D435 & D435i meshes to get rid of realsense2_description dependency

File: urdf/_d435.urdf.xacro (robot description, xacro)
@@ -66,7 +66,5 @@
       <origin xyz="${d435_cam_mount_from_center_offset} ${-d435_cam_depth_py} 0" rpy="${M_PI/2} 0 ${M_PI/2}"/>
         <geometry>
-          <!-- <box size="${d435_cam_width} ${d435_cam_height} ${d435_cam_depth}"/> -->
-          <mesh filename="package://realsense2_description/meshes/d435.dae"/>
-          <!--<mesh filename="package://realsense2_description/meshes/d435/d435.dae"/>-->
+          <mesh filename="package://realsense_gazebo_description/meshes/d435.dae"/>
         </geometry>
         <material name="${name}_aluminum"/>

File: urdf/_d435i.urdf.xacro (robot description, xacro)
@@ -69,7 +69,5 @@
       <origin xyz="${d435i_cam_mount_from_center_offset} ${-d435i_cam_depth_py} 0" rpy="${M_PI/2} 0 ${M_PI/2}"/>
         <geometry>
-          <!-- <box size="${d435i_cam_width} ${d435i_cam_height} ${d435i_cam_depth}"/> -->
-          <mesh filename="package://realsense2_description/meshes/d435.dae"/>
-          <!--<mesh filename="package://realsense2_description/meshes/d435/d435.dae"/>-->
+          <mesh filename="package://realsense_gazebo_description/meshes/d435.dae"/>
         </geometry>
         <material name="${name}_aluminum"/>

Commit message: Revert "Add D435 & D435i meshes to get rid of realsense2_description dependency"
This reverts commit 890e967773b170458df767070b3140d61e6773b8.

File: urdf/_d435.urdf.xacro (robot description, xacro)
@@ -66,5 +66,7 @@
       <origin xyz="${d435_cam_mount_from_center_offset} ${-d435_cam_depth_py} 0" rpy="${M_PI/2} 0 ${M_PI/2}"/>
         <geometry>
-          <mesh filename="package://realsense_gazebo_description/meshes/d435.dae"/>
+          <!-- <box size="${d435_cam_width} ${d435_cam_height} ${d435_cam_depth}"/> -->
+          <mesh filename="package://realsense2_description/meshes/d435.dae"/>
+          <!--<mesh filename="package://realsense2_description/meshes/d435/d435.dae"/>-->
         </geometry>
         <material name="${name}_aluminum"/>

File: urdf/_d435i.urdf.xacro (robot description, xacro)
@@ -69,5 +69,7 @@
       <origin xyz="${d435i_cam_mount_from_center_offset} ${-d435i_cam_depth_py} 0" rpy="${M_PI/2} 0 ${M_PI/2}"/>
         <geometry>
-          <mesh filename="package://realsense_gazebo_description/meshes/d435.dae"/>
+          <!-- <box size="${d435i_cam_width} ${d435i_cam_height} ${d435i_cam_depth}"/> -->
+          <mesh filename="package://realsense2_description/meshes/d435.dae"/>
+          <!--<mesh filename="package://realsense2_description/meshes/d435/d435.dae"/>-->
         </geometry>
         <material name="${name}_aluminum"/>
